File: voltmeter_module.kicad_sch (KiCad schematic)
At the start: 3 parts, among them U1 MCP3561RT-E_ST, U2 REF5050ID, U3 NCS20074D

Commit message: To je to otp
Parts:
- removed U2: REF5050ID, Package_SO:SOIC-8_3.9x4.9mm_P1.27mm, symbol Reference_Voltage:REF5050ID
- added K1: SANYOU_SRD_Form_A, Relay_THT:Relay_SPST_SANYOU_SRD_Series_Form_A, symbol Relay:SANYOU_SRD_Form_A
- added R1, R12, R13, R14, R15, R16, R17, R18, R19, R20: 1M, symbol Device:R_US
- added R10, R11, R2, R3, R4, R5, R6, R7, R8, R9: 24.9k, symbol Device:R_US
- added U2: TMUX1108PW, Package_SO:TSSOP-16_4.4x5mm_P0.65mm, symbol Analog_Switch:TMUX1108PW
- added U4: REF5030AD, Package_SO:SOIC-8_3.9x4.9mm_P1.27mm, symbol Reference_Voltage:REF5030AD
Connections:
- net ADC+: now reaches U3.1
- net ADC+: now also U1.5 (CH0), R6.2, U2.4 (S1)
- net at U3.2 (-): now also U2.8 (D)
- net at U3.3 (+): now also K1.3, R1.2
- net at U3.10 (+): now also R3.1, R4.2
- net INPUT-: now reaches U3.8
- net INPUT-: now also U1.6 (CH1), U3.9 (-), R2.1, R5.1, R9.1
- net +3.3V: now reaches U1.1 (AVDD)
- net +3.3V: now also U1.20 (DVDD), U4.2 (Vin)
- net GND: now reaches U1.19 (DGND)
- net GND: now also U1.2 (AGND), U1.3 (REFIN-), R4.1, U4.4 (GND)
- net 3V_ref: now reaches U1.4 (REFIN+/OUT)
- net 3V_ref: now also R3.2, U4.6 (Vout)
- new net: R7.1, R8.2, U2.6 (S3)
- new net: R6.1, R7.2, U2.5 (S2)
- new net: R16.1, R18.1
- new net: R15.1, R16.2
- new net: R12.1, R14.1
- new net: R13.1, R14.2
- new net: K1.1, R2.2, R5.2
- new net: R10.1, R11.2, U2.12 (S5)
- new net: R10.2, R8.1, U2.7 (S4)
- new net: R1.1, R12.2
- new net: R17.2, R19.1
- new net: R19.2, R20.2
- new net: R11.1, R9.2, U2.11 (S6)
- new net: R13.2, R15.2
- new net: R18.2, R20.1
- new net INPUT+: R17.1
- no-connect marks 0 -> 6
Other:
- note added: "sets_to_middle"
- moved on the sheet: U3A, U3B, U3C, U3D, U3E

Commit message: Add millivolt input.
Parts:
- removed U2: TMUX1108PW, Package_SO:TSSOP-16_4.4x5mm_P0.65mm, symbol Analog_Switch:TMUX1108PW
- added U5: ISO7762FDW, Package_SO:SOIC-16W_7.5x10.3mm_P1.27mm, symbol Isolator:ISO7762FDW
- added U6: 4051, Package_SO:SOIC-16_3.9x9.9mm_P1.27mm, symbol 4xxx:4051
Connections:
- net +3.3V: now also U5.16 (Vcc2), U6.16 (VDD)
- net ADC+: now also U6.13 (X0)
- net GND: now also U5.9 (GND2), U6.7 (VEE), U6.8 (VSS)
- net at R7.1, R8.2: now also U6.15 (X2)
- net at R6.1, R7.2: now also U6.14 (X1)
- net at U3.2 (-): now also U6.3 (X)
- net MV_INPUT+: now reaches K1.3, R1.2, U3.3 (+)
- net at R10.1, R11.2: now also U6.1 (X4)
- net at R10.2, R8.1: now also U6.12 (X3)
- net at R11.1, R9.2: now also U6.5 (X5)
- net at U1.13 (~{CS}): now also U5.14 (OUTB)
- net at U1.14 (SCK): now also U5.13 (OUTC)
- net at U1.15 (SDI): now also U5.12 (OUTD)
- net at U1.16 (SDO): now also U5.10 (INF)
- net at U1.18 (MCLK): now also U5.15 (OUTA)
Other:
- moved on the sheet: R1, R12, R13, R14, R15, R16, R17, R18, R19, R20, R3, R4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

Commit message: Tex.
Other:
- note added: "USE TELECOM PUSH PULL TRANSFORMER FOR POWER SUPPLY"
Changed lines of the file:
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@@
+		)
+	)
+	(text_box "10 Meg || 12.5 k \n12 k, 450 fA/Hz\n5.4 nV/Hz, less\nthan the voltage \nnoise"
+		(exclude_from_sim no)
+		(at 97.79 83.82 0)
+		(size 12.7 19.05)
+		(stroke
+			(width 0)
+			(type default)
+		)
+		(fill
+			(type color)
+			(color 62 129 255 1)
+		)
+		(effects
+			(font
+				(size 1.27 1.27)
+				(color 255 4 0 1)
+			)
+			(justify left top)
 		)
 	)
@@
 			)
 		)
+	)
+	(text "USE TELECOM PUSH PULL TRANSFORMER FOR POWER SUPPLY"
+		(exclude_from_sim no)
+		(at 260.858 87.122 0)
+		(effects
+			(font
+				(size 5.08 5.08)
+			)
+		)

Commit message: TL072 for the win.
Parts:
- removed K1: SANYOU_SRD_Form_A, Relay_THT:Relay_SPST_SANYOU_SRD_Series_Form_A, symbol Relay:SANYOU_SRD_Form_A
- removed R1, R12, R13, R14, R15, R16, R17, R18, R19, R20: 1M, symbol Device:R_US
- removed R10, R11, R2, R3, R4, R5, R6, R7, R8, R9: 24.9k, symbol Device:R_US
- removed U1: MCP3561RT-E_ST, Package_SO:TSSOP-20_4.4x6.5mm_P0.65mm, symbol rack_modules:MCP3561RT-E_ST
- removed U3: NCS20074D, Package_SO:SOIC-14_3.9x8.7mm_P1.27mm, symbol Amplifier_Operational:NCS20074D
- removed U4: REF5030AD, Package_SO:SOIC-8_3.9x4.9mm_P1.27mm, symbol Reference_Voltage:REF5030AD
- removed U5: ISO7762FDW, Package_SO:SOIC-16W_7.5x10.3mm_P1.27mm, symbol Isolator:ISO7762FDW
- removed U6: 4051, Package_SO:SOIC-16_3.9x9.9mm_P1.27mm, symbol 4xxx:4051
Connections:
- no-connect marks 6 -> 0
Other:
- added sheet Digital section (digital_section.kicad_sch)
- added sheet Input stage (input_stage.kicad_sch)
- added sheet Power supply (power_supply.kicad_sch)
- note removed: "Napravi baterija modul za kalibracioni modul"
- note removed: "Napravi kalibracioni modul"
- note removed: "USE TELECOM PUSH PULL TRANSFORMER FOR POWER SUPPLY"
- note removed: "sets_to_middle"
- note removed: "verzioniši module po rezoluciji, 4.5 ima lm4040, 5.5 ima ref5050, 6.5 ima lm399 itd"
