File: input_stage.kicad_sch (KiCad schematic)
At the start: 62 parts, among them K1 EE2-3NUX, Q1 2N7002, U1 REF5030AD, U2 TL072, U4 TL072, U6 NCS21802DMR2G, U7 CD4051B

Commit message: fixed resistor
Parts:
- R19, R21, R39, R40, R41, R42, R43, R44, R45, R6: value 100k -> 10k
Changed lines of the file:
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@@
 			)
 		)
-		(property "Value" "100k"
+		(property "Value" "10k"
 			(at 72.644 58.42 90)
 			(effects
@@
 			)
 		)
-		(property "Value" "100k"
+		(property "Value" "10k"
 			(at 72.644 48.26 90)
 			(effects
@@
 			)
 		)
-		(property "Value" "100k"
+		(property "Value" "10k"
 			(at 82.804 48.26 90)
 			(effects
@@
 			)
 		)
-		(property "Value" "100k"
+		(property "Value" "10k"
 			(at 72.644 38.1 90)
 			(effects
@@
 			)
 		)
-		(property "Value" "100k"
+		(property "Value" "10k"
 			(at 82.804 38.1 90)
 			(effects
@@
 			)
 		)
-		(property "Value" "100k"
+		(property "Value" "10k"
 			(at 82.804 29.21 90)
 			(effects
@@
 			)
 		)
-		(property "Value" "100k"
+		(property "Value" "10k"
 			(at 72.644 29.21 90)
 			(effects
@@
 			)
 		)
-		(property "Value" "100k"
+		(property "Value" "10k"
 			(at 82.804 58.42 90)
 			(effects
@@
 			)
 		)
-		(property "Value" "100k"
+		(property "Value" "10k"
 			(at 44.196 29.21 90)
 			(effects
@@
 			)
 		)
-		(property "Value" "100k"
+		(property "Value" "10k"
 			(at 54.356 29.21 90)
 			(effects

Commit message: Bootstraped input buffer.
Parts:
- removed U2: TL072, symbol Amplifier_Operational:TL072
- added C1, C10, C13, C14, C15, C2, C8, C9: 100n, Capacitor_SMD:C_0603_1608Metric_Pad1.08x0.95mm_HandSolder, symbol Device:C
- added C11, C12: 1u, Capacitor_SMD:C_0603_1608Metric_Pad1.08x0.95mm_HandSolder, symbol Device:C
- added D3, D4: ZF2V4, Diode_THT:D_DO-35_SOD27_P7.62mm_Horizontal, symbol Diode:BZV55B2V4
- added D5: BAT48ZFILM, Diode_SMD:D_SOD-123, symbol Diode:BAT48ZFILM
- added Q3, Q6, Q8: MMBT3904, Package_TO_SOT_SMD:SOT-23, symbol Transistor_BJT:MMBT3904
- added Q4, Q5, Q7: MMBT3906, Package_TO_SOT_SMD:SOT-23, symbol Transistor_BJT:MMBT3906
- added R53: 10, Resistor_SMD:R_0603_1608Metric_Pad0.98x0.95mm_HandSolder, symbol Device:R_US
- added R54, R55: 100, Resistor_SMD:R_0603_1608Metric_Pad0.98x0.95mm_HandSolder, symbol Device:R_US
- added R56, R57: 470, Resistor_SMD:R_0603_1608Metric_Pad0.98x0.95mm_HandSolder, symbol Device:R_US
- added R58: 100k, Resistor_SMD:R_0603_1608Metric_Pad0.98x0.95mm_HandSolder, symbol Device:R_US
- added U2: NCS21802DMR2G, Package_SO:OnSemi_Micro8, symbol voltmeter_lib:NCS21802DMR2G
Connections:
- net +3.3V: now also C10.2, C11.2, C2.2, D5.1 (K); no longer U1.2 (Vin)
- net -1V: now also C8.2
- net GND: now also C10.1, C11.1, C12.1, C13.1, C14.1, C15.1, C2.1, C8.1
- net BUFFER_OUT: now reaches R18.2
- net BUFFER_OUT: now also D3.1 (K), D4.2 (A), U2.1, U2.2 (-)
- net at K1.4, K1.9: now also R53.2, U2.3 (+)
- net at R51.2: now also U2.6 (-), U2.7
- net at K1.12, R15.2: now also D5.2 (A)
- net +15V renamed +15.3V
- net +15.3V: now also U1.2 (Vin), C12.2, C13.2, C14.2, Q3.3 (C), R54.2, R56.2
- net -15V renamed -15.3V
- net -15.3V: now also C15.2, Q4.3 (C), R55.1, R57.1
- new net: Q6.2 (E), R55.2
- new net: Q5.1 (B), Q7.1 (B), Q7.3 (C), R58.2
- new net: Q7.2 (E), R56.1
- new net: D4.1 (K), Q3.1 (B), Q5.3 (C)
- new net: C1.2, C9.2, Q3.2 (E), U2.8 (V+)
- new net: C1.1, C9.1, Q4.2 (E), U2.4 (V-)
- new net: R53.1, U2.5 (+)
- new net: Q6.1 (B), Q8.1 (B)
- new net: D3.2 (A), Q4.1 (B), Q6.3 (C)
- new net: Q5.2 (E), R54.1
- new net: Q8.2 (E), R57.2
- new net: Q8.3 (C), R58.1
Other:
- note added: "Input buffer bootstrap"
- moved on the sheet: Q1, R14, R15, R29
